File: hardware/esp32-s2-dev.kicad_pcb (KiCad board)
At the start: 2 copper layers, 23.4 x 45.4 mm, 31 parts, among them J1 USB_C_Receptacle_USB2.0_14P, J5 Conn_01x15, J6 Conn_01x15, SW1 SW_Push, U1 ESP32-S2, U2 XC6206PxxxMR, Y1 25MHz 20pF

Commit message: Update
Parts:
- added H2: MountingHole, logic-analyzer:Icy Electronics Logo, B.Cu at (160.1, 135.8)
